Commit message: Changed if condition and some other changes in process_image.cpp and remove duplicate model

File: my_robot/urdf/my_robot.xacro (robot description, xacro)
@@ -180,5 +180,5 @@
 	</gazebo>
   <gazebo reference="chassis">
-    <material>Gazebo/Black</material>
+    <material>Gazebo/Pink</material>
   </gazebo>
   <gazebo reference="camera">

Commit message: SLAM Project

File: my_robot/urdf/my_robot.xacro (robot description, xacro)
@@ -67,4 +67,11 @@
     <axis xyz="0.0 1.0 0.0"/>
   </joint>
+  <joint name="camera_optical_joint" type="fixed">
+    <origin xyz="0 0 0" rpy="-1.5707 0 -1.5707"/>
+    <parent link="camera"/>
+    <child link="camera_link_optical"/>
+  </joint>
+  <link name="camera_link_optical">
+  </link>
   <link name="left_wheel">
     <inertial>
@@ -173,15 +180,3 @@
     </visual>
   </link>
-  <gazebo reference="left_wheel">
-    <material>Gazebo/Red</material>
-	</gazebo>
-  <gazebo reference="right_wheel">
-    <material>Gazebo/Red</material>
-	</gazebo>
-  <gazebo reference="chassis">
-    <material>Gazebo/Pink</material>
-  </gazebo>
-  <gazebo reference="camera">
-    <material>Gazebo/Green</material>
-  </gazebo>
 </robot>
